File: src/rp2350_devboard.kicad_sch (KiCad schematic)
At the start: 26 parts, among them J1 USB_C_Receptacle_USB2.0_14P, U1 RP2350_60QFN, U2 MCP1700x-330xxTT

Commit message: Schematic finished
Parts:
- added C18, C19: 15p, symbol Device:C
- added C20: 100n, symbol Device:C
- added J2, J3: Conn_01x20, symbol Connector_Generic:Conn_01x20
- added J4: Conn_01x03, symbol Connector_Generic:Conn_01x03
- added R6, R8, R9: 1k, symbol Device:R
- added R7: 10k, symbol Device:R
- added SW1, SW2: SW_Push, symbol Switch:SW_Push
- added U3: W25Q128JVS, Package_SO:SOIC-8_5.3x5.3mm_P1.27mm, symbol Memory_Flash:W25Q128JVS
- added Y1: 12 MHz( ABM8-272-T3), symbol Device:Crystal_GND24
Connections:
- net +3.3V: now also C20.1, J3.5 (Pin_5), R7.1, U3.8 (VCC)
- net GND: now also C18.2, C19.2, C20.2, J2.13 (Pin_13), J2.18 (Pin_18), J2.3 (Pin_3), J2.8 (Pin_8), J3.13 (Pin_13), J3.18 (Pin_18), J3.3 (Pin_3), J3.8 (Pin_8), J4.2 (Pin_2), SW1.1, SW2.1, U3.4 (GND), Y1.2, Y1.4
- net VBUS: now also J3.1 (Pin_1)
- net GPIO7: now reaches U1.10 (GPIO7)
- net GPIO7: now also J2.10 (Pin_10)
- net GPIO8: now reaches U1.12 (GPIO8)
- net GPIO8: now also J2.11 (Pin_11)
- net GPIO9: now reaches U1.13 (GPIO9)
- net GPIO9: now also J2.12 (Pin_12)
- net GPIO10: now reaches U1.14 (GPIO10)
- net GPIO10: now also J2.14 (Pin_14)
- net GPIO11: now reaches U1.15 (GPIO11)
- net GPIO11: now also J2.15 (Pin_15)
- net GPIO12: now reaches U1.16 (GPIO12)
- net GPIO12: now also J2.16 (Pin_16)
- net GPIO13: now reaches U1.17 (GPIO13)
- net GPIO13: now also J2.17 (Pin_17)
- net GPIO14: now reaches U1.18 (GPIO14)
- net GPIO14: now also J2.19 (Pin_19)
- net GPIO15: now reaches U1.19 (GPIO15)
- net GPIO15: now also J2.20 (Pin_20)
- net GPIO0: now reaches U1.2 (GPIO0)
- net GPIO0: now also J2.1 (Pin_1)
- net XIN: now reaches U1.21 (XIN)
- net XIN: now also C18.1, Y1.1
- net XOUT: now reaches U1.22 (XOUT)
- net XOUT: now also R6.2
- net SWCLK: now reaches U1.24 (SWCLK)
- net SWCLK: now also J4.1 (Pin_1)
- net SWD: now reaches U1.25 (SWD)
- net SWD: now also J4.3 (Pin_3)
- net RUN: now reaches U1.26 (RUN)
- net RUN: now also J3.11 (Pin_11), R9.2
- net GPIO16: now reaches U1.27 (GPIO16)
- net GPIO16: now also J3.20 (Pin_20)
- net GPIO17: now reaches U1.28 (GPIO17)
- net GPIO17: now also J3.19 (Pin_19)
- net GPIO18: now reaches U1.29 (GPIO18)
- net GPIO18: now also J3.17 (Pin_17)
- net GPIO1: now reaches U1.3 (GPIO1)
- net GPIO1: now also J2.2 (Pin_2)
- net GPIO19: now reaches U1.31 (GPIO19)
- net GPIO19: now also J3.16 (Pin_16)
- net GPIO20: now reaches U1.32 (GPIO20)
- net GPIO20: now also J3.15 (Pin_15)
- net GPIO21: now reaches U1.33 (GPIO21)
- net GPIO21: now also J3.14 (Pin_14)
- net GPIO22: now reaches U1.34 (GPIO22)
- net GPIO22: now also J3.12 (Pin_12)
- net GPIO23: now reaches U1.35 (GPIO23)
- net GPIO23: now also J3.10 (Pin_10)
- net GPIO24: now reaches U1.36 (GPIO24)
- net GPIO24: now also J3.9 (Pin_9)
- net GPIO2: now reaches U1.4 (GPIO2)
- net GPIO2: now also J2.4 (Pin_4)
- net GPIO26_ADC0: now reaches U1.40 (GPIO26_ADC0)
- net GPIO26_ADC0: now also J3.7 (Pin_7)
- net GPIO27_ADC1: now reaches U1.41 (GPIO27_ADC1)
- net GPIO27_ADC1: now also J3.6 (Pin_6)
- net GPIO28_ADC2: now reaches U1.42 (GPIO28_ADC2)
- net GPIO28_ADC2: now also J3.4 (Pin_4)
- net GPIO29_ADC3: now reaches U1.43 (GPIO29_ADC3)
- net GPIO29_ADC3: now also J3.2 (Pin_2)
- net GPIO3: now reaches U1.5 (GPIO3)
- net GPIO3: now also J2.5 (Pin_5)
- net QSPI_SD3: now reaches U1.55 (QSPI_SD3)
- net QSPI_SD3: now also U3.7 (~{HOLD}/~{RESET}/IO_{3})
- net QSPI_SCLK: now reaches U1.56 (QSPI_SCLK)
- net QSPI_SCLK: now also U3.6 (CLK)
- net QSPI_SD0: now reaches U1.57 (QSPI_SD0)
- net QSPI_SD0: now also U3.5 (DI/IO_{0})
- net QSPI_SD2: now reaches U1.58 (QSPI_SD2)
- net QSPI_SD2: now also U3.3 (~{WP}/IO_{2})
- net QSPI_SD1: now reaches U1.59 (QSPI_SD1)
- net QSPI_SD1: now also U3.2 (DO/IO_{1})
- net QSPI_SS: now reaches U1.60 (QSPI_SS)
- net QSPI_SS: now also R7.2, R8.2, U3.1 (~{CS})
- net GPIO4: now reaches U1.7 (GPIO4)
- net GPIO4: now also J2.6 (Pin_6)
- net GPIO5: now reaches U1.8 (GPIO5)
- net GPIO5: now also J2.7 (Pin_7)
- net GPIO6: now reaches U1.9 (GPIO6)
- net GPIO6: now also J2.9 (Pin_9)
- new net: R9.1, SW2.2
- new net: C19.1, R6.1, Y1.3
- new net: R8.1, SW1.2
- no-connect marks 0 -> 1
Other:
- moved on the sheet: C1, C10, C11, C12, C13, C14, C15, C16, C17, C2, C3, C4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

Commit message: Assigned all footprints
Parts:
- C1, C10, C11, C12, C13, C14, C15, C18, C19, C2, C20, C3, C4, C5, C6, C7, C8, C9: footprint (none) -> Capacitor_SMD:C_0402_1005Metric
- C16, C17: footprint (none) -> Capacitor_SMD:C_0603_1608Metric
- J1: footprint (none) -> Connector_USB:USB_C_Receptacle_HRO_TYPE-C-31-M-12
- J2, J3: footprint (none) -> Connector_PinHeader_2.54mm:PinHeader_1x20_P2.54mm_Vertical
- J4: footprint (none) -> Connector_PinHeader_2.54mm:PinHeader_1x03_P2.54mm_Vertical
- L1: footprint (none) -> RP2350_60QFN_minimal:L_pol_2016
- R1, R2, R3, R4, R5, R6, R7, R8, R9: footprint (none) -> Resistor_SMD:R_0402_1005Metric
- SW1, SW2: footprint (none) -> Button_Switch_SMD:SW_Push_SPST_NO_Alps_SKRK
- Y1: value 12 MHz( ABM8-272-T3) -> 12 MHz; footprint (none) -> Crystal:Crystal_SMD_3225-4Pin_3.2x2.5mm
Other:
- note added: "ABM8-272-T3"
Changed lines of the file:
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@@
 		(date "2025-10-04")
 	)
+	(text "ABM8-272-T3"
+		(exclude_from_sim no)
+		(at 67.818 212.344 0)
+		(effects
+			(font
+				(size 1.27 1.27)
+			)
+		)
+	)
 	(text_box "Flash Memory"
 		(exclude_from_sim no)
@@
 			)
 		)
-		(property "Footprint" ""
+		(property "Footprint" "Resistor_SMD:R_0402_1005Metric"
 			(at 66.04 60.198 90)
 			(effects
@@
 			)
 		)
-		(property "Footprint" ""
+		(property "Footprint" "Resistor_SMD:R_0402_1005Metric"
 			(at 158.75 76.708 90)
 			(effects
@@
 			)
 		)
-		(property "Footprint" ""
+		(property "Footprint" "Connector_PinHeader_2.54mm:PinHeader_1x20_P2.54mm_Vertical"
 			(at 337.82 127 0)
 			(effects
@@
 			)
 		)
-		(property "Footprint" ""
+		(property "Footprint" "Capacitor_SMD:C_0402_1005Metric"
 			(at 91.44 137.4648 0)
 			(effects
@@
 			)
 		)
-		(property "Footprint" ""
+		(property "Footprint" "Resistor_SMD:R_0402_1005Metric"
 			(at 49.022 139.7 90)
 			(effects
@@
 			)
 		)
-		(property "Footprint" ""
+		(property "Footprint" "Connector_USB:USB_C_Receptacle_HRO_TYPE-C-31-M-12"
 			(at 48.26 68.58 0)
 			(effects
@@
 			)
 		)
-		(property "Footprint" ""
+		(property "Footprint" "Capacitor_SMD:C_0402_1005Metric"
 			(at 262.5852 62.23 0)
 			(effects
@@
 			)
 		)
-		(property "Footprint" ""
+		(property "Footprint" "Button_Switch_SMD:SW_Push_SPST_NO_Alps_SKRK"
 			(at 341.63 193.04 0)
 			(effects
@@
 			)
 		)
-		(property "Footprint" ""
+		(property "Footprint" "Capacitor_SMD:C_0402_1005Metric"
 			(at 239.7252 62.23 0)
 			(effects
@@
 			)
 		)
-		(property "Footprint" ""
+		(property "Footprint" "Resistor_SMD:R_0402_1005Metric"
 			(at 254 88.138 90)
 			(effects
@@
 			)
 		)
-		(property "Footprint" ""
+		(property "Footprint" "RP2350_60QFN_minimal:L_pol_2016"
 			(at 154.94 91.44 0)
 			(effects
@@
 			)
 		)
-		(property "Footprint" ""
+		(property "Footprint" "Connector_PinHeader_2.54mm:PinHeader_1x03_P2.54mm_Vertical"
 			(at 351.79 153.67 0)
 			(effects
@@
 			)
 		)
-		(property "Footprint" ""
+		(property "Footprint" "Capacitor_SMD:C_0603_1608Metric"
 			(at 82.2452 62.23 0)
 			(effects
@@
 			)
 		)
-		(property "Footprint" ""
+		(property "Footprint" "Capacitor_SMD:C_0402_1005Metric"
 			(at 308.3052 62.23 0)
 			(effects
@@
 			)
 		)
-		(property "Footprint" ""
+		(property "Footprint" "Capacitor_SMD:C_0402_1005Metric"
 			(at 251.1552 62.23 0)
 			(effects
@@
 			)
 		)
-		(property "Footprint" ""
+		(property "Footprint" "Capacitor_SMD:C_0603_1608Metric"
 			(at 102.5652 62.23 0)
 			(effects
@@
 			)
 		)
-		(property "Footprint" ""
+		(property "Footprint" "Resistor_SMD:R_0402_1005Metric"
 			(at 78.74 226.822 90)
 			(effects
@@
 			)
 		)
-		(property "Footprint" ""
+		(property "Footprint" "Resistor_SMD:R_0402_1005Metric"
 			(at 254 87.122 90)
 			(effects
@@
 			)
 		)
-		(property "Footprint" ""
+		(property "Footprint" "Resistor_SMD:R_0402_1005Metric"
 			(at 44.45 147.828 90)
 			(effects
@@
 			)
 		)
-		(property "Value" "12 MHz( ABM8-272-T3)"
+		(property "Value" "12 MHz"
 			(at 67.564 214.376 90)
 			(effects
@@
 			)
 		)
-		(property "Footprint" ""
+		(property "Footprint" "Crystal:Crystal_SMD_3225-4Pin_3.2x2.5mm"
 			(at 67.31 222.25 0)
 			(effects
@@
 			)
 		)
-		(property "Footprint" ""
+		(property "Footprint" "Capacitor_SMD:C_0402_1005Metric"
 			(at 46.99 229.5652 0)
 			(effects
@@
 			)
 		)
-		(property "Footprint" ""
+		(property "Footprint" "Capacitor_SMD:C_0402_1005Metric"
 			(at 319.7352 62.23 0)
 			(effects
@@
 			)
 		)
-		(property "Footprint" ""
+		(property "Footprint" "Capacitor_SMD:C_0402_1005Metric"
 			(at 274.0152 62.23 0)
 			(effects
@@
 			)
 		)
-		(property "Footprint" ""
+		(property "Footprint" "Capacitor_SMD:C_0402_1005Metric"
 			(at 183.8452 55.88 0)
 			(effects
@@
 			)
 		)
-		(property "Footprint" ""
+		(property "Footprint" "Capacitor_SMD:C_0402_1005Metric"
 			(at 172.4152 55.88 0)
 			(effects
@@
 			)
 		)
-		(property "Footprint" ""
+		(property "Footprint" "Capacitor_SMD:C_0402_1005Metric"
 			(at 143.2052 96.52 0)
 			(effects
@@
 			)
 		)
-		(property "Footprint" ""
+		(property "Footprint" "Capacitor_SMD:C_0402_1005Metric"
 			(at 331.1652 62.23 0)
 			(effects
@@
 			)
 		)
-		(property "Footprint" ""
+		(property "Footprint" "Capacitor_SMD:C_0402_1005Metric"
 			(at 169.8752 85.09 0)
 			(effects
@@
 			)
 		)
-		(property "Footprint" ""
+		(property "Footprint" "Capacitor_SMD:C_0402_1005Metric"
 			(at 131.7752 96.52 0)
 			(effects
@@
 			)
 		)
-		(property "Footprint" ""
+		(property "Footprint" "Capacitor_SMD:C_0402_1005Metric"
 			(at 46.99 218.1352 0)
 			(effects
@@
 			)
 		)
-		(property "Footprint" ""
+		(property "Footprint" "Resistor_SMD:R_0402_1005Metric"
 			(at 66.04 59.182 90)
 			(effects
@@
 			)
 		)
-		(property "Footprint" ""
+		(property "Footprint" "Resistor_SMD:R_0402_1005Metric"
 			(at 353.06 199.898 90)
 			(effects
@@
 			)
 		)
-		(property "Footprint" ""
+		(property "Footprint" "Capacitor_SMD:C_0402_1005Metric"
 			(at 160.9852 55.88 0)
 			(effects
@@
 			)
 		)
-		(property "Footprint" ""
+		(property "Footprint" "Button_Switch_SMD:SW_Push_SPST_NO_Alps_SKRK"
 			(at 33.02 140.97 0)
 			(effects
@@
 			)
 		)
-		(property "Footprint" ""
+		(property "Footprint" "Capacitor_SMD:C_0402_1005Metric"
 			(at 296.8752 62.23 0)
 			(effects
@@
 			)
 		)
-		(property "Footprint" ""
+		(property "Footprint" "Capacitor_SMD:C_0402_1005Metric"
 			(at 285.4452 62.23 0)
 			(effects
@@
 			)
 		)
-		(property "Footprint" ""
+		(property "Footprint" "Connector_PinHeader_2.54mm:PinHeader_1x20_P2.54mm_Vertical"
 			(at 364.49 127 0)
 			(effects
